File: blender/3d circuits/Hbridge/hbridge1.brd (EAGLE design)
At the start: 13 parts, among them Q2 IRLML0060, Q3 IRLML0060, Q4 IRLML0060, Q5 IRLML0060

Commit message: 3d circuit design
Parts:
- moved Q3 15.0 mm to (76.3, 21.8), flipped to the bottom, turned to 225 degrees
- moved D4 14.9 mm to (77.2, 29.1), turned to 315 degrees
- moved R1 11.7 mm to (69.2, 13.6), turned to 270 degrees
- moved Q2 10.3 mm to (77.0, 25.3), flipped to the bottom, turned to 45 degrees
- moved JP2 9.86 mm to (71.4, 27.3), turned to 45 degrees
- moved R7 8.31 mm to (71.6, 22.4), turned to 270 degrees
- moved JP1 8.21 mm to (59.4, 16.0)
- moved D5 3.69 mm to (65.9, 16.5), turned to 0 degrees
- moved Q4 3.44 mm to (74.1, 19.7), turned to 315 degrees
- moved D3 2.57 mm to (77.2, 34.8), turned to 45 degrees
- moved JP4 2.29 mm to (82.5, 30.5)
- moved Q5 0.75 mm to (70.0, 19.7), flipped to the bottom, turned to 315 degrees
Routing:
- net GND: track 39.1 -> 15.8 mm
- net VCC: track 28.4 -> 7.80 mm, vias 0 -> 1
- net COILA1: track 40.1 -> 35.2 mm, vias 0 -> 2
- net COILA2: track 9.48 -> 13.9 mm, vias 0 -> 1
- net GATEA1: track 18.4 -> 17.8 mm, vias 0 -> 1
- net GATEA2: track 36.7 -> 37.2 mm, vias 3 -> 1
