File: blender/3d circuits/Hbridge/hbridge1.sch (EAGLE design)
At the start: 13 parts, among them Q2 IRLML0060, Q3 IRLML0060, Q4 IRLML0060, Q5 IRLML0060

Commit message: 3d circuit design
Other:
- moved on the sheet: JP4
Changed lines of the file:
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@@
 <setting verticaltext="up"/>
 </settings>
-<grid distance="0.01" unitdist="inch" unit="inch" style="lines" multiple="1" display="yes" altdistance="0.01" altunitdist="inch" altunit="inch"/>
+<grid distance="0.1" unitdist="inch" unit="inch" style="lines" multiple="1" display="no" altdistance="0.01" altunitdist="inch" altunit="inch"/>
 <layers>
 <layer number="1" name="Top" color="4" fill="1" visible="no" active="no"/>
@@
 <instance part="FRAME1" gate="G$1" x="0" y="0"/>
 <instance part="P+4" gate="VCC" x="101.6" y="44.958"/>
-<instance part="JP4" gate="G$1" x="148.336" y="48.26" rot="R180"/>
+<instance part="JP4" gate="G$1" x="150.876" y="50.8" rot="R180"/>
 <instance part="Q2" gate="G$1" x="96.52" y="15.24"/>
 <instance part="D2" gate="G$1" x="101.6" y="15.24" rot="R90"/>
@@
 </segment>
 <segment>
-<wire x1="140.716" y1="48.26" x2="134.366" y2="48.26" width="0.1524" layer="91"/>
+<wire x1="143.256" y1="50.8" x2="134.366" y2="48.26" width="0.1524" layer="91"/>
 <pinref part="JP4" gate="G$1" pin="1"/>
 <label x="139.7" y="50.546" size="1.778" layer="95" rot="R180"/>
@@
 </segment>
 <segment>
-<wire x1="134.366" y1="45.72" x2="140.716" y2="45.72" width="0.1524" layer="91"/>
+<wire x1="131.826" y1="43.18" x2="143.256" y2="48.26" width="0.1524" layer="91"/>
 <pinref part="JP4" gate="G$1" pin="2"/>
 <label x="140.462" y="45.466" size="1.778" layer="95" rot="R180"/>
