File: blender/3d circuits/opamp/opampStone-v1.brd (EAGLE design)
At the start: 13 parts, among them Q2 IRLML0060, Q3 IRLML0060, Q4 IRLML0060, Q5 IRLML0060

Commit message: 3d circuit design
Parts:
- removed D2, D3, D4, D5: (no value), diode:DO-214AC
- removed Q2, Q3, Q4, Q5: IRLML0060, spietz-library:SOT-23
- removed R1, R7: 10K, resistor:R0603
- added JP3, JP6: M01PTH, SparkFun-Connectors:1X01
- added R12, R13: 1M, SparkFun-Passives:0805
- added R4, R8: 10k, SparkFun-Resistors:0603-RES
- added R5, R6: 10K, resistor:R0603
- added U2: MCP6242, spietz-library:8-SOIC
- moved JP4 75.6 mm to (14.2, 5.59)
- moved JP2 35.3 mm to (32.3, 5.59), turned to 270 degrees
- moved JP1 28.3 mm to (26.5, 20.6), turned to 0 degrees
Connections:
- removed net COILA1: D2.C, D4.A, JP4.1, Q2.3, Q4.2
- removed net COILA2: D3.A, D5.C, JP4.2, Q3.2, Q5.3
- removed net GATEA1: JP1.2, Q4.1, Q5.1, R7.2
- removed net GATEA2: JP1.1, Q2.1, Q3.1, R1.2
- new net A4: JP6.1, R13.2, U2.7
- new net A5: JP3.1, R12.2, U2.1
- new net MIDV: JP1.2, JP2.1, R5.1, R6.2, U2.3, U2.5
- new net N$13: R12.1, R4.2, U2.2
- new net N$15: R13.1, R8.2, U2.6
- new net SENSECOIL: JP2.2, R8.1
- new net SENSECOIL2: JP1.1, R4.1
- net GND: now also JP4.2, R6.1, U2.4; no longer D2.A, D5.A, JP2.1, Q2.2, Q5.2, R1.1, R7.1
- net VCC: now also JP4.1, R5.2, U2.8; no longer D3.C, D4.C, JP2.2, Q3.3, Q4.3
Routing:
- net MIDV: track 0.00 -> 79.0 mm
- net GND: track 0.00 -> 10.5 mm
- net VCC: track 0.00 -> 5.37 mm
Other:
- board text added: "10k"
- board text added: "1M"
- board text added: "CoilA"
- board text added: "Vcc"
- board text added: "coilB"
- board text added: "outA"
- board text added: "outB"
- board text removed: "+"
- board text removed: "coil"
- board text removed: "driveA1"
- board text removed: "driveA2"
